Commit message: urdf with meshes

File: description/materials.xacro (robot description, xacro)
@@ -13,3 +13,6 @@
     <color rgba="0 0 0 1"/>
 </material>
+<material name="gray">
+    <color rgba="0.5 0.5 0.5 1"/>
+</material>
 </robot>

File: description/robot_core.xacro (robot description, xacro)
@@ -4,25 +4,26 @@
     <xacro:include filename="inertial_macros.xacro"/>
     <link name="base_link">
+        <origin xyz="0 0 0.01"/>
     </link>
     <joint name="chassis_joint" type="fixed">
         <parent link="base_link"/>
         <child link="chassis"/>
-        <origin xyz="-0.1 0 0"/>
+        <origin xyz="0 0 0.0023" rpy="0 0 ${pi}"/>
     </joint>
     <link name="chassis">
         <visual>
-            <origin xyz="0.15 0 0.075"/>
+            <origin xyz="0 0 0"/>
             <geometry>
-                <box size="0.3 0.3 0.15"/>
+                <mesh filename="package://pg1_project/description/meshes/BODY.stl" scale="0.001 0.001 0.001"/>
             </geometry>
             <material name="red"/>
         </visual>
         <collision>
-            <origin xyz="0.15 0 0.075"/>
+            <origin xyz="-0.13 0 0.1"/>
             <geometry>
-                <box size="0.3 0.3 0.15"/>
+                <box size="0.4 0.5 0.3"/>
             </geometry>
         </collision>
-        <xacro:inertial_box mass="0.5" x="0.3" y="0.3" z="0.15">
+        <xacro:inertial_box mass="4" x="0.4" y="0.3" z="0.2">
             <origin xyz="0.15 0 0.075" rpy="0 0 0"/>
         </xacro:inertial_box>
@@ -31,5 +32,5 @@
         <parent link="base_link"/>
         <child link="left_wheel"/>
-        <origin xyz="0 0.175 0" rpy="-${pi/2} 0 0"/>
+        <origin xyz="0 0.2 0" rpy="-${pi/2} 0 0"/>
         <axis xyz="0 0 1"/>
     </joint>
@@ -37,14 +38,14 @@
         <visual>
             <geometry>
-                <cylinder radius="0.05" length="0.04"/>
+                <mesh filename="package://pg1_project/description/meshes/WHEEL.stl" scale="0.001 0.001 0.001"/>
             </geometry>
-            <material name="black"/>
+            <material name="gray"/>
         </visual>
         <collision>
             <geometry>
-                <cylinder radius="0.05" length="0.04"/>
+                <mesh filename="package://pg1_project/description/meshes/WHEEL.stl" scale="0.001 0.001 0.001"/>
             </geometry>
         </collision>
-        <xacro:inertial_cylinder mass="0.1" radius="0.05" length="0.04">
+        <xacro:inertial_cylinder mass="3" radius="0.16" length="0.04">
             <origin xyz="0 0 0" rpy="0 0 0"/>
         </xacro:inertial_cylinder>
@@ -53,5 +54,5 @@
         <parent link="base_link"/>
         <child link="right_wheel"/>
-        <origin xyz="0 -0.175 0" rpy="${pi/2} 0 0"/>
+        <origin xyz="0 -0.2 0" rpy="${pi/2} 0 0"/>
         <axis xyz="0 0 -1"/>
     </joint>
@@ -59,14 +60,14 @@
         <visual>
             <geometry>
-                <cylinder radius="0.05" length="0.04"/>
+                <mesh filename="package://pg1_project/description/meshes/WHEEL.stl" scale="0.001 0.001 0.001"/>
             </geometry>
-            <material name="black"/>
+            <material name="gray"/>
         </visual>
         <collision>
             <geometry>
-                <cylinder radius="0.05" length="0.04"/>
+                <mesh filename="package://pg1_project/description/meshes/WHEEL.stl" scale="0.001 0.001 0.001"/>
             </geometry>
         </collision>
-        <xacro:inertial_cylinder mass="0.1" radius="0.05" length="0.04">
+        <xacro:inertial_cylinder mass="3" radius="0.16" length="0.04">
             <origin xyz="0 0 0" rpy="0 0 0"/>
         </xacro:inertial_cylinder>
@@ -75,16 +76,16 @@
         <parent link="base_link"/>
         <child link="caster_wheel"/>
-        <origin xyz="0.14 0 0" />
+        <origin xyz="0.31 0 -0.04" />
     </joint>
     <link name="caster_wheel">
         <visual>
             <geometry>
-                <sphere radius="0.05"/>
+                <cylinder radius="0.02" length="0.07"/>
             </geometry>
-            <material name="black"/>
+            <material name="gray"/>
         </visual>
         <collision>
             <geometry>
-                <sphere radius="0.05"/>
+                <cylinder radius="0.04" length="0.05"/>
             </geometry>
         </collision>
