Commit message: -

File: description/robot_core_with_meshes.xacro (robot description, xacro)
@@ -13,18 +13,18 @@
     <link name="chassis">
         <visual>
-            <origin xyz="-0.16 0 0.12"/>
+            <origin xyz="0 0 0"/>
             <geometry>
-                <box size="0.5 0.4 0.3"/>
+                <mesh filename="package://pg1_project/description/meshes/BODY.stl" scale="0.001 0.001 0.001"/>
             </geometry>
             <material name="red"/>
         </visual>
         <collision>
-            <origin xyz="-0.16 0 0.12"/>
+            <origin xyz="-0.13 0 0.1"/>
             <geometry>
-                <box size="0.5 0.4 0.3"/>
+                <box size="0.4 0.5 0.3"/>
             </geometry>
         </collision>
-        <xacro:inertial_box mass="4" x="0.5" y="0.4" z="0.3">
-            <origin xyz="-0.16 0 0.12" rpy="0 0 0"/>
+        <xacro:inertial_box mass="4" x="0.4" y="0.3" z="0.2">
+            <origin xyz="0.15 0 0.075" rpy="0 0 0"/>
         </xacro:inertial_box>
     </link>
@@ -38,5 +38,5 @@
         <visual>
             <geometry>
-                <cylinder radius="0.08" length="0.04"/>
+                <mesh filename="package://pg1_project/description/meshes/WHEEL.stl" scale="0.001 0.001 0.001"/>
             </geometry>
             <material name="gray"/>
@@ -44,8 +44,8 @@
         <collision>
             <geometry>
-                <cylinder radius="0.08" length="0.04"/>
+                <mesh filename="package://pg1_project/description/meshes/WHEEL.stl" scale="0.001 0.001 0.001"/>
             </geometry>
         </collision>
-        <xacro:inertial_cylinder mass="3" radius="0.08" length="0.04">
+        <xacro:inertial_cylinder mass="3" radius="0.16" length="0.04">
             <origin xyz="0 0 0" rpy="0 0 0"/>
         </xacro:inertial_cylinder>
@@ -60,5 +60,5 @@
         <visual>
             <geometry>
-                <cylinder radius="0.08" length="0.04"/>
+                <mesh filename="package://pg1_project/description/meshes/WHEEL.stl" scale="0.001 0.001 0.001"/>
             </geometry>
             <material name="gray"/>
@@ -66,8 +66,8 @@
         <collision>
             <geometry>
-                <cylinder radius="0.08" length="0.04"/>
+                <mesh filename="package://pg1_project/description/meshes/WHEEL.stl" scale="0.001 0.001 0.001"/>
             </geometry>
         </collision>
-        <xacro:inertial_cylinder mass="3" radius="0.08" length="0.04">
+        <xacro:inertial_cylinder mass="3" radius="0.16" length="0.04">
             <origin xyz="0 0 0" rpy="0 0 0"/>
         </xacro:inertial_cylinder>
@@ -81,5 +81,5 @@
         <visual>
             <geometry>
-                <cylinder radius="0.04" length="0.07"/>
+                <cylinder radius="0.02" length="0.07"/>
             </geometry>
             <material name="gray"/>
