Commit message: odrive

File: description/gazebo_control.xacro (robot description, xacro)
@@ -7,5 +7,5 @@
             <right_joint>right_wheel_joint</right_joint>
             <wheel_separation>0.4</wheel_separation>
-            <wheel_diameter>0.16</wheel_diameter>
+            <wheel_diameter>0.17</wheel_diameter>
             <!-- limits -->
             <max_wheel_torque>200</max_wheel_torque>

File: description/lidar.xacro (robot description, xacro)
@@ -4,5 +4,5 @@
         <parent link="base_link"/>
         <child link="laser_frame"/>
-        <origin xyz="0 0 0.3"/>
+        <origin xyz="0 0 0.3"  rpy="0 0 ${pi}"/>
     </joint>
     <link name="laser_frame">

File: description/robot_real.urdf.xacro (robot description, xacro)
@@ -3,5 +3,4 @@
     <!-- Example link -->
     <xacro:include filename="robot_core.xacro"/>
-    <xacro:include filename="gazebo_control.xacro"/>
     <xacro:include filename="lidar.xacro"/>
     <xacro:include filename="camera.xacro"/>
