Commit message: save

File: description/robot.urdf.xacro (robot description, xacro)
@@ -3,3 +3,4 @@
     <!-- Example link -->
     <xacro:include filename="robot_core.xacro"/>
+    <xacro:include filename="gazebo_control.xacro"/>
 </robot>

File: description/robot_core.xacro (robot description, xacro)
@@ -29,4 +29,7 @@
         </xacro:inertial_box>
     </link>
+    <gazebo reference="chassis">
+        <material>Gazebo/Red</material>
+    </gazebo>
     <joint name="left_wheel_joint" type="continuous">
         <parent link="base_link"/>
@@ -51,4 +54,7 @@
         </xacro:inertial_cylinder>
     </link>
+    <gazebo reference="left_wheel">
+        <material>Gazebo/Black</material>
+    </gazebo>
     <joint name="right_wheel_joint" type="continuous">
         <parent link="base_link"/>
@@ -73,8 +79,11 @@
         </xacro:inertial_cylinder>
     </link>
+    <gazebo reference="right_wheel">
+        <material>Gazebo/Black</material>
+    </gazebo>
     <joint name="caster_wheel_joint" type="fixed">
         <parent link="base_link"/>
         <child link="caster_wheel"/>
-        <origin xyz="0.31 0 -0.04" />
+        <origin xyz="0.31 0 -0.055" />
     </joint>
     <link name="caster_wheel">
@@ -94,3 +103,8 @@
         </xacro:inertial_sphere>
     </link>
+    <gazebo reference="caster_wheel">
+        <material>Gazebo/Black</material>
+        <mu1 value="0.001"/>
+        <mu2 value="0.001"/>
+    </gazebo>
 </robot>

Commit message: ros2 control

File: description/robot.urdf.xacro (robot description, xacro)
@@ -3,4 +3,6 @@
     <!-- Example link -->
     <xacro:include filename="robot_core.xacro"/>
-    <xacro:include filename="gazebo_control.xacro"/>
+    <!-- <xacro:include filename="gazebo_control.xacro"/> -->
+    <xacro:include filename="ros2_control.xacro"/>
+    <xacro:include filename="lidar.xacro"/>
 </robot>

File: description/robot_core.xacro (robot description, xacro)
@@ -9,5 +9,5 @@
         <parent link="base_link"/>
         <child link="chassis"/>
-        <origin xyz="0 0 0.0023" rpy="0 0 ${pi}"/>
+        <origin xyz="0 0 0.0023" rpy="0 0 0"/>
     </joint>
     <link name="chassis">
@@ -47,5 +47,5 @@
         <collision>
             <geometry>
-                <cylinder radius="0.08" length="0.04"/>
+                <sphere radius="0.08"/>
             </geometry>
         </collision>
@@ -72,5 +72,5 @@
         <collision>
             <geometry>
-                <cylinder radius="0.08" length="0.04"/>
+                <sphere radius="0.08" />
             </geometry>
         </collision>
@@ -85,5 +85,5 @@
         <parent link="base_link"/>
         <child link="caster_wheel"/>
-        <origin xyz="0.31 0 -0.055" />
+        <origin xyz="-0.31 0 -0.055" />
     </joint>
     <link name="caster_wheel">

Commit message: hardw int second try

File: description/robot.urdf.xacro (robot description, xacro)
@@ -3,5 +3,6 @@
     <!-- Example link -->
     <xacro:include filename="robot_core.xacro"/>
-    <xacro:include filename="gazebo_control.xacro"/>
+    <xacro:include filename="ros2_control.xacro"/>
+    <!-- <xacro:include filename="gazebo_control.xacro"/>  -->
     <xacro:include filename="lidar.xacro"/>
     <xacro:include filename="camera.xacro"/>

File: description/ros2_control.xacro (robot description, xacro)
@@ -1,5 +1,6 @@
 <?xml version="1.0"?>
 <robot xmlns:xacro="http://www.ros.org/wiki/xacro"  name="robot">
-    <!-- <ros2_control name="GazeboSystem" type="system">
+<!--
+    <ros2_control name="GazeboSystem" type="system">
         <hardware>
             <plugin>gazebo_ros2_control/GazeboSystem</plugin>
@@ -23,35 +24,22 @@
     </ros2_control> -->
     <ros2_control name="RealRobot" type="system">
-        <hardware>
-            <plugin>diffdrive_arduino/DiffDriveArduino</plugin>
-            <param name="left_wheel_name">left_wheel_joint</param>
-            <param name="right_wheel_name">right_wheel_joint</param>
-            <param name="loop_rate">30</param>
-            <param name="device">/dev/ttyUSB0</param>
-            <param name="baud_rate">57600</param>
-            <param name="timeout">1000</param>
-            <param name="enc_counts_per_rev">60</param>
-        </hardware>
+    <hardware>
+        <plugin>odrive_hardware_interface/ODriveHardwareInterface</plugin>
+    </hardware>
+    <sensor name="odrv0">
+        <param name="serial_number">123</param>
+    </sensor>
+        <joint name="right_wheel_joint">
+            <param name="serial_number">123</param>
+            <param name="axis">0</param>
+            <param name="enable_watchdog">1</param>
+            <param name="watchdog_timeout">0.1</param>
+        </joint>
         <joint name="left_wheel_joint">
-            <command_interface name="velocity">
-                <param name="min">-30</param>
-                <param name="max">30</param>
-            </command_interface>
-            <state_interface name="velocity"/>
-            <state_interface name="position"/>
-        </joint>
-        <joint name="right_wheel_joint">
-            <command_interface name="velocity">
-                <param name="min">-30</param>
-                <param name="max">30</param>
-            </command_interface>
-            <state_interface name="velocity"/>
-            <state_interface name="position"/>
+            <param name="serial_number">123</param>
+            <param name="axis">1</param>
+            <param name="enable_watchdog">1</param>
+            <param name="watchdog_timeout">0.1</param>
         </joint>
     </ros2_control>
-    <gazebo>
-        <plugin name="gazebo_ros2_control" filename="libgazebo_ros2_control.so">
-            <parameters>/home/pgiust/dev_ws/src/pg1_project/config/my_controllers.yaml</parameters>
-        </plugin>
-    </gazebo>
 </robot>
