Commit message: navigation dev machine

File: description/lidar.xacro (robot description, xacro)
@@ -4,5 +4,5 @@
         <parent link="base_link"/>
         <child link="laser_frame"/>
-        <origin xyz="0 0 0.3"  rpy="0 0 ${pi}"/>
+        <origin xyz="0 0 0.31"  rpy="0 0 ${pi}"/>
     </joint>
     <link name="laser_frame">
@@ -12,4 +12,5 @@
             </geometry>
             <material name="black"/>
+            <origin xyz="0 0 0" rpy="0 0 0"/>
         </visual>
         <collision>
@@ -17,4 +18,5 @@
                 <cylinder radius="0.08" length="0.04"/>
             </geometry>
+            <origin xyz="0 0 0" rpy="0 0 0"/>
         </collision>
         <xacro:inertial_cylinder mass="3" radius="0.08" length="0.04">
@@ -26,5 +28,5 @@
         <sensor name="laser" type="ray">
             <pose> 0 0 0 0 0 0 </pose>
-            <visualize>false</visualize>
+            <visualize>true</visualize>
             <update_rate>10</update_rate>
             <ray>

File: description/ros2_control.xacro (robot description, xacro)
@@ -1,5 +1,5 @@
 <?xml version="1.0"?>
 <robot xmlns:xacro="http://www.ros.org/wiki/xacro"  name="robot">
-    <!-- <ros2_control name="GazeboSystem" type="system">
+    <ros2_control name="GazeboSystem" type="system">
         <hardware>
             <plugin>gazebo_ros2_control/GazeboSystem</plugin>
@@ -26,6 +26,6 @@
             <parameters>$(find pg1_project)/config/my_controllers_sim.yaml</parameters>
         </plugin>
-    </gazebo> -->
-    <ros2_control name="RealRobot" type="system">
+    </gazebo>
+    <!-- <ros2_control name="RealRobot" type="system">
     <hardware>
         <plugin>odrive_hardware_interface/ODriveHardwareInterface</plugin>
@@ -46,4 +46,4 @@
             <param name="watchdog_timeout">0.1</param>
         </joint>
-    </ros2_control>
+    </ros2_control> -->
 </robot>
