Commit message: save2

File: description/camera.xacro (robot description, xacro)
@@ -4,5 +4,5 @@
         <parent link="chassis"/>
         <child link="camera_link"/>
-        <origin xyz="0.10 0 0.25" rpy="0 0 0"/>
+        <origin xyz="0.10 0 0.14" rpy="0 0 0"/>
     </joint>
     <link name="camera_link">

File: description/lidar.xacro (robot description, xacro)
@@ -4,10 +4,10 @@
         <parent link="base_link"/>
         <child link="laser_frame"/>
-        <origin xyz="0 0 0.31"  rpy="0 0 ${pi}"/>
+        <origin xyz="0.05 0 0.20"  rpy="0 0 ${pi}"/>
     </joint>
     <link name="laser_frame">
         <visual>
             <geometry>
-                <cylinder radius="0.08" length="0.04"/>
+                <cylinder radius="0.04" length="0.04"/>
             </geometry>
             <material name="black"/>

File: description/robot_core.xacro (robot description, xacro)
@@ -20,7 +20,7 @@
     <link name="chassis">
         <visual>
-            <origin xyz="-0.16 0 0.12"/>
+            <origin xyz="-0.13 0 0.09"/>
             <geometry>
-                <box size="0.5 0.4 0.3"/>
+                <box size="0.42 0.36 0.2"/>
             </geometry>
             <material name="red"/>
@@ -92,10 +92,10 @@
         <parent link="base_link"/>
         <child link="caster_wheel"/>
-        <origin xyz="-0.31 0 -0.055" />
+        <origin xyz="-0.28 0 -0.045" />
     </joint>
     <link name="caster_wheel">
         <visual>
             <geometry>
-                <cylinder radius="0.04" length="0.07"/>
+                <cylinder radius="0.04" length="0.09"/>
             </geometry>
             <material name="gray"/>
