Commit message: frontback camera

File: description/camera_back.xacro (robot description, xacro)
@@ -1,10 +1,10 @@
 <?xml version="1.0"?>
 <robot xmlns:xacro="http://www.ros.org/wiki/xacro" >
-    <joint name="camera_joint" type="fixed">
+    <joint name="camera_back_joint" type="fixed">
         <parent link="chassis"/>
-        <child link="camera_link"/>
-        <origin xyz="0.10 0 0.14" rpy="0 0 0"/>
+        <child link="camera_back_link"/>
+        <origin xyz="-0.35 0 0.1" rpy="0 0.2 0"/>
     </joint>
-    <link name="camera_link">
+    <link name="camera_back_link">
         <visual>
             <geometry>
@@ -14,13 +14,13 @@
         </visual>
     </link>
-    <joint name="camera_optical_joint" type="fixed">
-        <parent link="camera_link"/>
-        <child link="camera_link_optical"/>
+    <joint name="camera_back_optical_joint" type="fixed">
+        <parent link="camera_back_link"/>
+        <child link="camera_back_link_optical"/>
         <origin xyz="0 0 0" rpy="${-pi/2} 0 ${-pi/2}"/>
     </joint>
-    <link name="camera_link_optical"></link>
-    <gazebo reference="camera_link">
+    <link name="camera_back_link_optical"></link>
+    <gazebo reference="camera_back_link">
         <material>Gazebo/Black</material>
-        <sensor name="camera" type="camera">
+        <sensor name="camera_back" type="camera">
             <pose> 0 0 0 0 0 0 </pose>
             <visualize>true</visualize>

File: description/robot.urdf.xacro (robot description, xacro)
@@ -6,4 +6,5 @@
     <!-- <xacro:include filename="gazebo_control.xacro"/>  -->
     <xacro:include filename="lidar.xacro"/>
-    <xacro:include filename="camera.xacro"/>
+    <xacro:include filename="camera_front.xacro"/>
+    <xacro:include filename="camera_back.xacro"/>
 </robot>

Commit message: df

File: description/camera_back.xacro (robot description, xacro)
@@ -4,5 +4,5 @@
         <parent link="chassis"/>
         <child link="camera_back_link"/>
-        <origin xyz="-0.35 0 0.1" rpy="0 0.2 0"/>
+        <origin xyz="-0.35 0 0.1" rpy="0 -0.2 ${pi}"/>
     </joint>
     <link name="camera_back_link">
@@ -38,5 +38,5 @@
                 </clip>
             </camera>
-            <plugin name="camera_controller" filename="libgazebo_ros_camera.so">
+            <plugin name="camera_back_controller" filename="libgazebo_ros_camera.so">
                 <frame_name>camera_link_optical</frame_name>
             </plugin>

File: description/camera_front.xacro (robot description, xacro)
@@ -38,5 +38,5 @@
                 </clip>
             </camera>
-            <plugin name="camera_controller" filename="libgazebo_ros_camera.so">
+            <plugin name="camera_front_controller" filename="libgazebo_ros_camera.so">
                 <frame_name>camera_link_optical</frame_name>
             </plugin>
