Commit message: sim now works

File: description/robot_core.xacro (robot description, xacro)
@@ -41,5 +41,5 @@
         <visual>
             <geometry>
-                <cylinder radius="0.08" length="0.04"/>
+                <cylinder radius="0.085" length="0.04"/>
             </geometry>
             <material name="gray"/>
@@ -47,8 +47,8 @@
         <collision>
             <geometry>
-                <sphere radius="0.08"/>
+                <sphere radius="0.085"/>
             </geometry>
         </collision>
-        <xacro:inertial_cylinder mass="3" radius="0.08" length="0.04">
+        <xacro:inertial_cylinder mass="3" radius="0.085" length="0.04">
             <origin xyz="0 0 0" rpy="0 0 0"/>
         </xacro:inertial_cylinder>
@@ -66,5 +66,5 @@
         <visual>
             <geometry>
-                <cylinder radius="0.08" length="0.04"/>
+                <cylinder radius="0.085" length="0.04"/>
             </geometry>
             <material name="gray"/>
@@ -72,8 +72,8 @@
         <collision>
             <geometry>
-                <sphere radius="0.08" />
+                <sphere radius="0.085" />
             </geometry>
         </collision>
-        <xacro:inertial_cylinder mass="3" radius="0.08" length="0.04">
+        <xacro:inertial_cylinder mass="3" radius="0.085" length="0.04">
             <origin xyz="0 0 0" rpy="0 0 0"/>
         </xacro:inertial_cylinder>

File: description/ros2_control.xacro (robot description, xacro)
@@ -1,5 +1,4 @@
 <?xml version="1.0"?>
 <robot xmlns:xacro="http://www.ros.org/wiki/xacro"  name="robot">
-<!--
     <ros2_control name="GazeboSystem" type="system">
         <hardware>
@@ -22,6 +21,11 @@
             <state_interface name="position"/>
         </joint>
-    </ros2_control> -->
-    <ros2_control name="RealRobot" type="system">
+    </ros2_control>
+    <gazebo>
+        <plugin name="gazebo_ros2_control" filename="libgazebo_ros2_control.so">
+            <parameters>$(find pg1_project)/config/my_controllers_sim.yaml</parameters>
+        </plugin>
+    </gazebo>
+    <!-- <ros2_control name="RealRobot" type="system">
     <hardware>
         <plugin>odrive_hardware_interface/ODriveHardwareInterface</plugin>
@@ -42,4 +46,4 @@
             <param name="watchdog_timeout">0.1</param>
         </joint>
-    </ros2_control>
+    </ros2_control> -->
 </robot>

Commit message: footprint

File: description/robot_core.xacro (robot description, xacro)
@@ -5,4 +5,11 @@
     <link name="base_link">
         <origin xyz="0 0 0.01"/>
+    </link>
+     <joint name="base_footprint_joint" type="fixed">
+        <parent link="base_link"/>
+        <child link="base_footprint"/>
+        <origin xyz="0 0 -0.01" rpy="0 0 0"/>
+    </joint>
+    <link name="base_footprint">
     </link>
     <joint name="chassis_joint" type="fixed">
@@ -19,10 +26,10 @@
             <material name="red"/>
         </visual>
-        <collision>
+        <!-- <collision>
             <origin xyz="-0.16 0 0.12"/>
             <geometry>
                 <box size="0.5 0.4 0.3"/>
             </geometry>
-        </collision>
+        </collision> -->
         <xacro:inertial_box mass="4" x="0.5" y="0.4" z="0.3">
             <origin xyz="-0.16 0 0.12" rpy="0 0 0"/>

Commit message: deployment code good

File: description/robot_core.xacro (robot description, xacro)
@@ -9,5 +9,5 @@
         <parent link="base_link"/>
         <child link="base_footprint"/>
-        <origin xyz="0 0 -0.01" rpy="0 0 0"/>
+        <origin xyz="-0.14 0 -0.01" rpy="0 0 0"/>
     </joint>
     <link name="base_footprint">

Commit message: hshs

File: description/robot_core.xacro (robot description, xacro)
@@ -103,5 +103,5 @@
         <collision>
             <geometry>
-                <cylinder radius="0.04" length="0.05"/>
+                <cylinder radius="0.04" length="0.08"/>
             </geometry>
         </collision>
